File: mekanisk-40 14U.kicad_sch (KiCad schematic)
At the start: 135 parts, among them J1 USB_C_Receptacle_USB2.0, Q1 2N7002, SW1 RST, U2 USBLC6-2SC6, U3 STM32F072C8Tx, U4 XC6206PxxxMR-Regulator_Linear

Commit message: created 13u & 14u keyboard versions
Parts:
- removed D47: D_Small, Diode_SMD:D_SOD-123F, symbol Device:D_Small
- removed MX40, MX47, MX48, MX49: MX_SW_HS, PCM_marbastlib-mx:SW_MX_1.5u, symbol PCM_marbastlib-mx:MX_SW_HS
- removed MX43: MX_SW_HS, PCM_marbastlib-mx:SW_MX_1u, symbol PCM_marbastlib-mx:MX_SW_HS
- added D48, D49, D50, D51: D_Small, Diode_SMD:D_SOD-123F, symbol Device:D_Small
- added MX50, MX51, MX52, MX53: MX_SW_HS, PCM_marbastlib-mx:SW_MX_1u, symbol PCM_marbastlib-mx:MX_SW_HS
- MX37, MX39, MX45, MX46: footprint PCM_marbastlib-mx:SW_MX_1u -> PCM_marbastlib-mx:SW_MX_1.25u
Connections:
- net COL11: now also MX50.1, MX51.1, MX52.1, MX53.1; no longer MX12.1, MX24.1, MX36.1, MX46.1, MXISO1.1, MXenter2.25.1, MXshift2.75.1
- net ROW0: now also D48.1 (K)
- net ROW1: now also D49.1 (K)
- net ROW2: now also D50.1 (K)
- net ROW3: now also D51.1 (K)
- net at D43.2 (A): now also MXsplit2.25.2
- new net: D48.2 (A), MX50.2
- new net: D50.2 (A), MX52.2
- new net: D51.2 (A), MX53.2
- new net: D49.2 (A), MX51.2
- new net COL12: MX12.1, MX24.1, MX36.1, MX46.1, MXISO1.1, MXenter2.25.1, MXshift2.75.1
Other:
- moved on the sheet: D12, D24, D36, D46, ISO1, MX12, MX24, MX36, MX46, MXISO1, MXenter2.25, MXshift2.75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
