File: mekanisk-40.kicad_pcb (KiCad board)
At the start: 2 copper layers, 247.7 x 76.2 mm, 132 parts, among them J2 USB_C_Receptacle_USB2.0, Q1 2N7002, SW1 RST, U1 USBLC6-2SC6, U2 XC6206PxxxMR-Regulator_Linear, U3 STM32F072C8Tx

Commit message: created 13u & 14u keyboard versions
Parts:
- added D40: D_Small, Diode_SMD:D_SOD-123F, B.Cu at (131.8, 97.6)
- added D47: D_Small, Diode_SMD:D_SOD-123F, B.Cu at (179.4, 97.6)
- added MX40: MX_SW_HS, PCM_marbastlib-mx:SW_MX_1.5u, F.Cu at (40.5, 98.4)
- added MX47: MX_SW_HS, PCM_marbastlib-mx:SW_MX_1.5u, F.Cu at (69.1, 98.4)
- added MX48: MX_SW_HS, PCM_marbastlib-mx:SW_MX_1.5u, F.Cu at (231.0, 98.4)
- added MX49: MX_SW_HS, PCM_marbastlib-mx:SW_MX_1.5u, F.Cu at (259.6, 98.4)
- added MXsplit2.25: MX_SW_HS, PCM_marbastlib-mx:SW_MX_1u, F.Cu at (176.2, 98.4)
- MX37, MX39, MX43, MX45: footprint PCM_marbastlib-mx:SW_MX_1.25u -> PCM_marbastlib-mx:SW_MX_1u
- S1: footprint PCM_marbastlib-mx:STAB_MX_P_6.25u -> PCM_marbastlib-mx:STAB_MX_P_7u
- moved ? 72.2 mm to (111.9, 129.4), turned to 180 degrees
- moved S2 61.9 mm to (176.2, 98.4)
- moved MXsplit2.75 33.3 mm to (128.6, 98.4)
- moved S3 33.3 mm to (128.6, 98.4)
- moved D41 21.4 mm to (96.0, 97.6)
- moved MX41 21.4 mm to (92.9, 98.4)
- moved ? 12.1 mm to (144.5, 129.4), turned to 180 degrees
- moved D42 11.9 mm to (153.2, 97.6)
- moved D44 9.53 mm to (234.2, 97.6)
- moved D43 7.14 mm to (210.3, 97.6)
- moved MX39 7.14 mm to (73.8, 98.4)
- moved D39 7.14 mm to (77.0, 97.6)
- moved MX43 7.14 mm to (207.2, 98.4)
- moved MX38 4.76 mm to (54.8, 98.4)
- moved D38 4.76 mm to (57.9, 97.6)
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Connections:
- MX41 pad 1: COL4 -> COL3
- MXsplit2.75 pad 1: COL6 -> COL5
- MXsplit2.75 pad 2: Net-(D42-A) -> Net-(D40-A)
Routing:
- net COL5: track 105.3 -> 127.3 mm
- net COL3: track 67.6 -> 88.6 mm
- net COL4: track 106.5 -> 86.4 mm
- net COL7: track 143.3 -> 163.3 mm
- net COL6: track 158.8 -> 148.5 mm
- net Net-(D42-A): track 12.7 -> 3.15 mm
- net COL9: track 205.9 -> 212.6 mm
- net COL2: track 68.9 -> 75.6 mm
- net GND: track 82.4 -> 88.6 mm, vias 10 -> 12
- net Net-(D44-A): track 3.15 -> 7.91 mm
- net Net-(D39-A): track 3.15 -> 7.91 mm
- net Net-(D37-A): track 3.15 -> 7.91 mm
- net Net-(D46-A): track 3.15 -> 7.91 mm
- net COL11: track 261.6 -> 266.3 mm
- net COL0: track 118.3 -> 123.0 mm
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Other:
- board text added: "1.5U"
- board text added: "1U"
- board text added: "7U"
- board text added: "mekanisk40 (13U)"
- board text removed: "6.25U"
- board text removed: "mekanisk40"

Commit message: changed routing and reset button placement on 13u
Parts:
- moved SW1 30.3 mm to (46.8, 68.3), turned to 90 degrees
- moved Q1 23.4 mm to (51.6, 70.8), turned to -90 degrees
- moved C11 22.9 mm to (51.6, 66.3), turned to 180 degrees
- moved R5 22.8 mm to (51.6, 67.9), turned to 0 degrees
- moved R3 18.1 mm to (51.6, 64.6), turned to 180 degrees
- moved C10 18.1 mm to (54.5, 69.7), turned to -90 degrees
- moved R4 15.9 mm to (56.1, 69.7), turned to -90 degrees
- moved D13 0.79 mm to (46.0, 60.3)
- moved D14 0.79 mm to (72.2, 60.3)
- moved D15 0.79 mm to (91.3, 60.3)
- moved D16 0.79 mm to (110.3, 60.3)
- moved D17 0.79 mm to (129.4, 60.3)
- moved D18 0.79 mm to (148.4, 60.3)
- moved D19 0.79 mm to (167.5, 60.3)
- moved D20 0.79 mm to (186.5, 60.3)
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Routing:
- net NRST: track 14.2 -> 27.2 mm, vias 0 -> 2
- net GND: track 88.6 -> 82.3 mm, vias 12 -> 10
- net +3V3: track 91.2 -> 96.8 mm, vias 6 -> 7
- net BOOT0: track 31.0 -> 35.7 mm
- net COL6: track 148.5 -> 145.1 mm
- net Net-(D36-A): track 12.7 -> 13.9 mm
- net Net-(D24-A): track 12.9 -> 14.1 mm
- net ROW3: track 475.0 -> 476.0 mm
- net ROW2: track 455.3 -> 456.3 mm, vias 2 -> 0
- net Net-(D46-A): track 7.91 -> 8.71 mm
- net Net-(D44-A): track 7.91 -> 8.71 mm
- net Net-(D39-A): track 7.91 -> 8.71 mm
- net Net-(D47-A): track 3.15 -> 3.94 mm
- net Net-(D45-A): track 3.15 -> 3.94 mm
- net Net-(D43-A): track 3.15 -> 3.94 mm
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
Commit message: minimal gnd fill, added jst pico footprints
Parts:
- added D_PWR1: SMF9.0CA, Diode_SMD:D_SOD-123, B.Cu at (56.4, 44.5)
- added J1: JST SH, Connector_JST:JST_SH_SM04B-SRSS-TB_1x04-1MP_P1.00mm_Horizontal, B.Cu at (62.7, 48.4)
- added J3: Pico EZmate, Connector_Molex:Molex_Pico-EZmate_78171-0004_1x04-1MP_P1.20mm_Vertical, B.Cu at (64.3, 48.4)
- turned R3 to 0 degrees
Routing:
- net GND: track 82.3 -> 174.4 mm, vias 10 -> 13
- net +5V: track 15.3 -> 34.7 mm, vias 0 -> 2
- net D_USB_N: track 6.62 -> 23.6 mm, vias 0 -> 2
- net D_USB_P: track 6.62 -> 20.3 mm, vias 0 -> 2
- net NRST: track 27.2 -> 33.5 mm
- net BOOT0: track 35.7 -> 34.5 mm
- removed copper zone on F.Cu, net GND
Other:
- board text added: "1"
- board text added: "1.25"
- board text added: "1.5"
- board text added: "1.75"
- board text added: "2.25"
- board text added: "2.75"
- board text added: "7"
- board text added: "ISO"
- board text added: "stepped"
- board text removed: "1.5U"
- board text removed: "1U"
- board text removed: "2.25U"
- board text removed: "2.75U"
- board text removed: "7U"

Commit message: update
Routing:
- net D_USB_N: track 23.6 -> 26.1 mm
- net D_USB_P: track 20.3 -> 21.8 mm
Changed lines of the file:
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@@
   (segment (start 60.570742 62.179456) (end 60.314393 61.923107) (width 0.381) (layer "B.Cu") (net 62))
   (segment (start 55.220458 52.989768) (end 55.220458 57.510959) (width 0.25) (layer "B.Cu") (net 62))
+  (segment (start 57.413204 42.740676) (end 57.35388 42.8) (width 0.25) (layer "B.Cu") (net 62))
   (segment (start 69.91899 76.73926) (end 69.21799 76.03826) (width 0.381) (layer "B.Cu") (net 62))
   (segment (start 57.18125 41.975) (end 57.18125 41.275) (width 0.25) (layer "B.Cu") (net 62))
@@
   (segment (start 56.375 52.96875) (end 55.241476 52.96875) (width 0.25) (layer "B.Cu") (net 62))
   (segment (start 73.81875 69.05625) (end 73.828096 69.065596) (width 0.25) (layer "B.Cu") (net 62))
-  (segment (start 57.35388 42.8) (end 56.35625 42.8) (width 0.25) (layer "B.Cu") (net 62))
   (segment (start 55.220458 57.510959) (end 59.632606 61.923107) (width 0.25) (layer "B.Cu") (net 62))
   (segment (start 53.140749 42.8625) (end 56.29375 42.8625) (width 0.25) (layer "B.Cu") (net 62))
@@
   (segment (start 69.84651 67.46526) (end 70.541453 66.770317) (width 0.2) (layer "B.Cu") (net 62))
   (segment (start 78.58125 69.83125) (end 79.35625 69.05625) (width 0.2) (layer "B.Cu") (net 62))
+  (segment (start 57.35388 42.8) (end 56.35625 42.8) (width 0.25) (layer "B.Cu") (net 62))
   (segment (start 57.18125 39.72) (end 55.6375 38.17625) (width 0.2) (layer "B.Cu") (net 62))
   (segment (start 56.29375 42.8625) (end 56.35625 42.8) (width 0.25) (layer "B.Cu") (net 62))
@@
   (segment (start 60.622742 64.591492) (end 62.845103 66.813853) (width 0.381) (layer "B.Cu") (net 62))
   (segment (start 69.85 70.634405) (end 70.829229 69.655176) (width 0.25) (layer "B.Cu") (net 62))
-  (segment (start 57.413204 42.740676) (end 57.35388 42.8) (width 0.25) (layer "B.Cu") (net 62))
   (segment (start 68.453851 63.389085) (end 66.977266 61.9125) (width 0.2) (layer "B.Cu") (net 62))
   (segment (start 69.201909 70.640483) (end 68.268578 70.640483) (width 0.25) (layer "B.Cu") (net 62))
@@
   (segment (start 51.1375 39.9175) (end 49.78 41.275) (width 0.25) (layer "B.Cu") (net 67))
   (segment (start 49.78 41.275) (end 49.24375 41.275) (width 0.25) (layer "B.Cu") (net 67))
-  (segment (start 54.743524 42.092014) (end 58.846681 46.195171) (width 0.25) (layer "F.Cu") (net 68))
-  (segment (start 58.846681 46.195171) (end 58.846681 48.91615) (width 0.25) (layer "F.Cu") (net 68))
+  (segment (start 57.15 44.49849) (end 57.125755 44.474245) (width 0.25) (layer "F.Cu") (net 68))
+  (segment (start 54.743524 42.092014) (end 57.125755 44.474245) (width 0.25) (layer "F.Cu") (net 68))
+  (segment (start 57.15 48.64325) (end 57.15 44.49849) (width 0.25) (layer "F.Cu") (net 68))
   (via (at 54.743524 42.092014) (size 0.8) (drill 0.4) (layers "F.Cu" "B.Cu") (net 68))
-  (via (at 58.846681 48.91615) (size 0.8) (drill 0.4) (layers "F.Cu" "B.Cu") (net 68))
+  (via (at 57.15 48.64325) (size 0.8) (drill 0.4) (layers "F.Cu" "B.Cu") (net 68))
+  (segment (start 58.846681 48.91615) (end 59.53125 48.91615) (width 0.25) (layer "B.Cu") (net 68))
   (segment (start 53.0875 37.15125) (end 53.1375 37.20125) (width 0.2) (layer "B.Cu") (net 68))
+  (segment (start 59.53125 48.91615) (end 60.70365 48.91615) (width 0.25) (layer "B.Cu") (net 68))
   (segment (start 52.1875 37.15125) (end 53.0875 37.15125) (width 0.2) (layer "B.Cu") (net 68))
   (segment (start 52.1375 38.17625) (end 52.1375 37.20125) (width 0.2) (layer "B.Cu") (net 68))
@@
   (segment (start 54.37651 41.725) (end 54.743524 42.092014) (width 0.25) (layer "B.Cu") (net 68))
   (segment (start 53.1375 41.525) (end 53.3375 41.725) (width 0.25) (layer "B.Cu") (net 68))
+  (segment (start 59.53125 48.91615) (end 57.4229 48.91615) (width 0.25) (layer "B.Cu") (net 68))
   (segment (start 60.70365 48.91615) (end 60.70625 48.91875) (width 0.25) (layer "B.Cu") (net 68))
   (segment (start 62.31875 48.91875) (end 60.70625 48.91875) (width 0.25) (layer "B.Cu") (net 68))
   (segment (start 62.41875 49.01875) (end 62.31875 48.91875) (width 0.25) (layer "B.Cu") (net 68))
   (segment (start 53.1375 37.20125) (end 53.1375 38.17625) (width 0.2) (layer "B.Cu") (net 68))
-  (segment (start 58.846681 48.91615) (end 60.70365 48.91615) (width 0.25) (layer "B.Cu") (net 68))
-  (segment (start 58.01051 46.561809) (end 53.340498 41.891797) (width 0.25) (layer "F.Cu") (net 69))
-  (segment (start 58.01051 47.927434) (end 58.01051 46.561809) (width 0.25) (layer "F.Cu") (net 69))
+  (segment (start 57.4229 48.91615) (end 57.15 48.64325) (width 0.25) (layer "B.Cu") (net 68))
+  (segment (start 55.829101 47.452853) (end 55.829101 44.380401) (width 0.25) (layer "F.Cu") (net 69))
+  (segment (start 54.539975 43.091275) (end 53.340498 41.891797) (width 0.25) (layer "F.Cu") (net 69))
   (segment (start 53.340498 41.891797) (end 50.166506 41.891797) (width 0.25) (layer "F.Cu") (net 69))
-  (via (at 58.01051 47.927434) (size 0.8) (drill 0.4) (layers "F.Cu" "B.Cu") (net 69))
+  (segment (start 55.829101 44.380401) (end 54.539975 43.091275) (width 0.25) (layer "F.Cu") (net 69))
   (via (at 50.166506 41.891797) (size 0.8) (drill 0.4) (layers "F.Cu" "B.Cu") (net 69))
+  (via (at 55.829101 47.452853) (size 0.8) (drill 0.4) (layers "F.Cu" "B.Cu") (net 69))
   (segment (start 62.41875 47.81875) (end 62.31875 47.91875) (width 0.25) (layer "B.Cu") (net 69))
   (segment (start 50.333303 41.725) (end 50.166506 41.891797) (width 0.25) (layer "B.Cu") (net 69))
   (segment (start 52.5875 39.20125) (end 51.6875 39.20125) (width 0.2) (layer "B.Cu") (net 69))
-  (segment (start 60.70625 47.91875) (end 58.019194 47.91875) (width 0.25) (layer "B.Cu") (net 69))
+  (segment (start 60.70625 47.91875) (end 59.53125 47.91875) (width 0.25) (layer "B.Cu") (net 69))
   (segment (start 51.6375 39.15125) (end 51.6375 38.17625) (width 0.2) (layer "B.Cu") (net 69))
   (segment (start 51.6375 41.525) (end 51.4375 41.725) (width 0.25) (layer "B.Cu") (net 69))
+  (segment (start 59.53125 47.91875) (end 56.294998 47.91875) (width 0.25) (layer "B.Cu") (net 69))
   (segment (start 62.31875 47.91875) (end 60.70625 47.91875) (width 0.25) (layer "B.Cu") (net 69))
   (segment (start 51.6375 38.17625) (end 51.6375 41.525) (width 0.25) (layer "B.Cu") (net 69))
+  (segment (start 56.294998 47.91875) (end 55.829101 47.452853) (width 0.25) (layer "B.Cu") (net 69))
   (segment (start 58.019194 47.91875) (end 58.01051 47.927434) (width 0.25) (layer "B.Cu") (net 69))
   (segment (start 52.6375 39.15125) (end 52.5875 39.20125) (width 0.2) (layer "B.Cu") (net 69))
+  (segment (start 59.53125 47.91875) (end 58.019194 47.91875) (width 0.25) (layer "B.Cu") (net 69))
   (segment (start 52.6375 38.17625) (end 52.6375 39.15125) (width 0.2) (layer "B.Cu") (net 69))
   (segment (start 51.6875 39.20125) (end 51.6375 39.15125) (width 0.2) (layer "B.Cu") (net 69))
@@
     (polygon
       (pts
-        (xy 59.258297 45.297365)
-        (xy 66.830797 45.255447)
+        (xy 59.22735 44.848849)
+        (xy 66.79985 44.806931)
         (xy 66.838771 52.028289)
         (xy 59.258296 52.086039)

Commit message: routing update
Routing:
- net GND: track 174.4 -> 175.9 mm

Commit message: backup
Other:
- board text added: "JLCJLCJLCJLC"
Changed lines of the file:
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@@
     (effects (font (size 1 1) (thickness 0.15)) (justify mirror))
+  )
+  (gr_text "JLCJLCJLCJLC" (at 52.3875 33.3375) (layer "B.SilkS")
+    (effects (font (size 1 1) (thickness 0.15)))
   )
   (gr_text "2.25" (at 48.41875 83.34375) (layer "B.SilkS")

Commit message: slight routing change, necessary?
Parts:
- C10: value 1u -> 1uF
- C11: value 4.7u -> 4.7uF
- moved C7 0.78 mm to (78.6, 68.3)
- moved C9 0.77 mm to (78.6, 69.9)
Connections:
- U3 pad 10: unconnected-(U3-PA0-Pad10) -> COL5
- U3 pad 11: unconnected-(U3-PA1-Pad11) -> COL4
- U3 pad 12: unconnected-(U3-PA2-Pad12) -> COL3
- U3 pad 13: unconnected-(U3-PA3-Pad13) -> COL2
- U3 pad 2: COL6 -> unconnected-(U3-PC13-Pad2)
- U3 pad 3: COL5 -> unconnected-(U3-PC14-Pad3)
- U3 pad 38: ROW0 -> unconnected-(U3-PA15-Pad38)
- U3 pad 39: ROW3 -> ROW0
- U3 pad 4: COL4 -> unconnected-(U3-PC15-Pad4)
- U3 pad 40: ROW2 -> ROW3
- U3 pad 41: COL11 -> ROW2
- U3 pad 42: COL10 -> COL11
- U3 pad 43: COL9 -> COL10
- U3 pad 45: COL8 -> COL9
- U3 pad 46: COL7 -> COL8
- U3 pad 5: COL3 -> COL7
- U3 pad 6: COL2 -> COL6
Routing:
- net COL5: track 127.3 -> 130.7 mm
- net COL3: track 88.6 -> 92.0 mm
- net COL4: track 86.4 -> 89.8 mm
- net COL2: track 75.6 -> 78.6 mm
- net COL6: track 145.1 -> 147.9 mm
- net COL7: track 163.5 -> 165.8 mm
- net +3V3: track 96.8 -> 98.4 mm
- net GND: track 175.9 -> 176.9 mm
