File: Project/mekanical.kicad_pcb (KiCad board)
At the start: 2 copper layers, 247.7 x 76.2 mm, 142 parts, among them J1 JST SH, J2 USB_C_Receptacle_USB2.0, J3 Pico EZmate, Q1 2N7002, SW1 RST, U1 USBLC6-2SC6, U2 XC6206PxxxMR-Regulator_Linear, U3 STM32F072C8Tx

Commit message: update
Other:
- board text added: "decide on mounting"
- board text added: "mekanical"
- board text removed: "mekanisk40 (13U)"
Changed lines of the file:
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@@
     (fp_arc (start 8.53125 -5.499999) (mid 8.677685 -5.853565) (end 9.03125 -5.999999)
       (stroke (width 0.05) (type solid)) (layer "Eco2.User"))
-    (fp_arc (start 9.03125 8.000001) (mid 8.677729 7.853537) (end 8.53125 7.500001)
+    (fp_arc (start 9.03125 8.000001) (mid 8.677693 7.853543) (end 8.53125 7.500001)
       (stroke (width 0.05) (type solid)) (layer "Eco2.User"))
-    (fp_arc (start 14.780039 -5.999999) (mid 15.133567 -5.853539) (end 15.280039 -5.499999)
+    (fp_arc (start 14.780039 -5.999999) (mid 15.133602 -5.853545) (end 15.280039 -5.499999)
       (stroke (width 0.05) (type solid)) (layer "Eco2.User"))
-    (fp_arc (start 15.28125 7.500001) (mid 15.134806 7.853571) (end 14.78125 8.000001)
+    (fp_arc (start 15.28125 7.500001) (mid 15.1348 7.853536) (end 14.78125 8.000001)
       (stroke (width 0.05) (type solid)) (layer "Eco2.User"))
     (pad "" thru_hole circle locked (at -11.90625 -6.985) (size 4 4) (drill 3.048) (layers "*.Cu" "B.Mask"))
@@
     (fp_arc (start 8.53125 -5.499999) (mid 8.677685 -5.853565) (end 9.03125 -5.999999)
       (stroke (width 0.05) (type solid)) (layer "Eco2.User"))
-    (fp_arc (start 9.03125 8.000001) (mid 8.677729 7.853537) (end 8.53125 7.500001)
+    (fp_arc (start 9.03125 8.000001) (mid 8.677693 7.853543) (end 8.53125 7.500001)
       (stroke (width 0.05) (type solid)) (layer "Eco2.User"))
-    (fp_arc (start 14.780039 -5.999999) (mid 15.133567 -5.853539) (end 15.280039 -5.499999)
+    (fp_arc (start 14.780039 -5.999999) (mid 15.133602 -5.853545) (end 15.280039 -5.499999)
       (stroke (width 0.05) (type solid)) (layer "Eco2.User"))
-    (fp_arc (start 15.28125 7.500001) (mid 15.134806 7.853571) (end 14.78125 8.000001)
+    (fp_arc (start 15.28125 7.500001) (mid 15.1348 7.853536) (end 14.78125 8.000001)
       (stroke (width 0.05) (type solid)) (layer "Eco2.User"))
     (pad "" thru_hole circle locked (at -11.90625 -6.985) (size 4 4) (drill 3.048) (layers "*.Cu" "B.Mask"))
@@
     (fp_arc (start 8.53125 -5.499999) (mid 8.677685 -5.853565) (end 9.03125 -5.999999)
       (stroke (width 0.05) (type solid)) (layer "Eco2.User"))
-    (fp_arc (start 9.03125 8.000001) (mid 8.677729 7.853537) (end 8.53125 7.500001)
+    (fp_arc (start 9.03125 8.000001) (mid 8.677693 7.853543) (end 8.53125 7.500001)
       (stroke (width 0.05) (type solid)) (layer "Eco2.User"))
-    (fp_arc (start 14.780039 -5.999999) (mid 15.133567 -5.853539) (end 15.280039 -5.499999)
+    (fp_arc (start 14.780039 -5.999999) (mid 15.133602 -5.853545) (end 15.280039 -5.499999)
       (stroke (width 0.05) (type solid)) (layer "Eco2.User"))
-    (fp_arc (start 15.28125 7.500001) (mid 15.134806 7.853571) (end 14.78125 8.000001)
+    (fp_arc (start 15.28125 7.500001) (mid 15.1348 7.853536) (end 14.78125 8.000001)
       (stroke (width 0.05) (type solid)) (layer "Eco2.User"))
     (pad "" thru_hole circle locked (at -11.90625 -6.985 180) (size 4 4) (drill 3.048) (layers "*.Cu" "B.Mask"))
@@
     (fp_arc (start 8.53125 -5.499999) (mid 8.677685 -5.853565) (end 9.03125 -5.999999)
       (stroke (width 0.05) (type solid)) (layer "Eco2.User"))
-    (fp_arc (start 9.03125 8.000001) (mid 8.677729 7.853537) (end 8.53125 7.500001)
+    (fp_arc (start 9.03125 8.000001) (mid 8.677693 7.853543) (end 8.53125 7.500001)
       (stroke (width 0.05) (type solid)) (layer "Eco2.User"))
-    (fp_arc (start 14.780039 -5.999999) (mid 15.133567 -5.853539) (end 15.280039 -5.499999)
+    (fp_arc (start 14.780039 -5.999999) (mid 15.133602 -5.853545) (end 15.280039 -5.499999)
       (stroke (width 0.05) (type solid)) (layer "Eco2.User"))
-    (fp_arc (start 15.28125 7.500001) (mid 15.134806 7.853571) (end 14.78125 8.000001)
+    (fp_arc (start 15.28125 7.500001) (mid 15.1348 7.853536) (end 14.78125 8.000001)
       (stroke (width 0.05) (type solid)) (layer "Eco2.User"))
     (pad "" thru_hole circle locked (at -11.90625 -6.985 180) (size 4 4) (drill 3.048) (layers "*.Cu" "B.Mask"))
@@
     (fp_arc (start 8.53125 -5.499999) (mid 8.677685 -5.853565) (end 9.03125 -5.999999)
       (stroke (width 0.05) (type solid)) (layer "Eco2.User"))
-    (fp_arc (start 9.03125 8.000001) (mid 8.677729 7.853537) (end 8.53125 7.500001)
+    (fp_arc (start 9.03125 8.000001) (mid 8.677693 7.853543) (end 8.53125 7.500001)
       (stroke (width 0.05) (type solid)) (layer "Eco2.User"))
-    (fp_arc (start 14.780039 -5.999999) (mid 15.133567 -5.853539) (end 15.280039 -5.499999)
+    (fp_arc (start 14.780039 -5.999999) (mid 15.133602 -5.853545) (end 15.280039 -5.499999)
       (stroke (width 0.05) (type solid)) (layer "Eco2.User"))
-    (fp_arc (start 15.28125 7.500001) (mid 15.134806 7.853571) (end 14.78125 8.000001)
+    (fp_arc (start 15.28125 7.500001) (mid 15.1348 7.853536) (end 14.78125 8.000001)
       (stroke (width 0.05) (type solid)) (layer "Eco2.User"))
     (pad "" thru_hole circle locked (at -11.90625 -6.985) (size 4 4) (drill 3.048) (layers "*.Cu" "B.Mask"))
@@
   (gr_line (start 26.19375 82.55) (end 29.99375 82.55)
     (stroke (width 0.2) (type default)) (layer "Edge.Cuts"))
+  (gr_text "decide on mounting" (at 126.20625 115.8875) (layer "F.Cu")
+    (effects (font (size 3 3) (thickness 0.3) bold) (justify left bottom))
+  )
   (gr_text "7" (at 150.01875 102.39375) (layer "B.SilkS")
     (effects (font (size 1 1) (thickness 0.15)) (justify mirror))
@@
     (effects (font (size 1 1) (thickness 0.15)) (justify mirror))
   )
-  (gr_text "1.25" (at 261.9375 64.29375) (layer "B.SilkS")
+  (gr_text "1.25" (at 261.9375 65.88125) (layer "B.SilkS")
     (effects (font (size 1 1) (thickness 0.15)) (justify mirror))
   )
@@
     (effects (font (size 1 1) (thickness 0.15)) (justify mirror))
   )
-  (gr_text "mekanisk40 (13U)" (at 149.225 69.05625) (layer "F.SilkS")
+  (gr_text "mekanical" (at 149.225 69.05625) (layer "F.SilkS")
     (effects (font (size 3 3) (thickness 0.15)))
   )
