File: Project/mekanical.kicad_sch (KiCad schematic)
At the start: 138 parts, among them J1 JST SH, J1 USB_C_Receptacle_USB2.0, J3 Pico EZmate, Q1 2N7002, SW1 RST, U2 USBLC6-2SC6, U3 STM32F072C8Tx, U4 XC6206PxxxMR-Regulator_Linear

Commit message: created production files
Parts:
- removed C10: 1uF, Capacitor_SMD:C_0603_1608Metric, symbol Device:C_Small
- removed C11: 4.7uF, Capacitor_SMD:C_0603_1608Metric, symbol Device:C_Small
- removed C_USBSHIELD1: 4.7nF, Capacitor_SMD:C_0603_1608Metric, symbol Device:C_Small
- removed J1: JST SH, Connector_JST:JST_SH_SM04B-SRSS-TB_1x04-1MP_P1.00mm_Horizontal, symbol Connector_Generic_MountingPin:Conn_01x04_MountingPin
- removed J3: Pico EZmate, Connector_Molex:Molex_Pico-EZmate_78171-0004_1x04-1MP_P1.20mm_Vertical, symbol Connector_Generic_MountingPin:Conn_01x04_MountingPin
- removed Q1: 2N7002, Package_TO_SOT_SMD:SOT-23, symbol Transistor_FET:2N7002
- removed R3, R4: 10k, Resistor_SMD:R_0603_1608Metric, symbol Device:R_Small
- removed R5: 100k, Resistor_SMD:R_0603_1608Metric, symbol Device:R_Small
- removed R_USBSHIELD1: 1M, Resistor_SMD:R_0603_1608Metric, symbol Device:R_Small
- removed SW1: RST, Button_Switch_SMD:SW_SPST_SKQG_WithoutStem, symbol Switch:SW_Push
- added C?: 100nF, Capacitor_SMD:C_0603_1608Metric, symbol Device:C_Small
- added MX50, MX51: MX_SW_HS, PCM_marbastlib-mx:SW_MX_1.5u, symbol PCM_marbastlib-mx:MX_SW_HS
- added MXsplit2.25(1)1, MXsplit2.75(1)1: MX_SW_HS, PCM_marbastlib-mx:SW_MX_1u, symbol PCM_marbastlib-mx:MX_SW_HS
- added R?: 10k, Resistor_SMD:R_0603_1608Metric, symbol Device:R_Small
- added S4: MX_stab, PCM_marbastlib-mx:STAB_MX_P_2.25u, symbol PCM_marbastlib-mx:MX_stab
- added S5: MX_stab, PCM_marbastlib-mx:STAB_MX_P_2.75u, symbol PCM_marbastlib-mx:MX_stab
- added SW?: SKQGABE010, Button_Switch_SMD:SW_SPST_SKQG_WithoutStem, symbol Switch:SW_Push
- MX40: footprint PCM_marbastlib-mx:SW_MX_1.5u -> PCM_marbastlib-mx:SW_MX_1.75u
- MX47: footprint PCM_marbastlib-mx:SW_MX_1.5u -> PCM_marbastlib-mx:SW_MX_1u
Connections:
- net +3V3: now also SW?.1
- net BOOT0: now also R?.1, SW?.2
- net COL0: now also MX48.1; no longer MX40.1
- net COL10: now also MX40.1, U3.42 (PB6); no longer U3.43 (PB7)
- net COL11: now also MX47.1, U3.41 (PB5), MX51.1; no longer MX49.1, U3.42 (PB6)
- net COL2: now also MX49.1, U3.6 (PF1); no longer MX47.1, U3.13 (PA3)
- net COL3: now also U3.5 (PF0); no longer U3.12 (PA2)
- net COL4: now also U3.4 (PC15); no longer U3.11 (PA1)
- net COL5: now also U3.3 (PC14), MXsplit2.25(1)1.1; no longer U3.10 (PA0)
- net COL6: now also U3.2 (PC13); no longer U3.6 (PF1)
- net COL7: now also U3.46 (PB9), MXsplit2.75(1)1.1; no longer U3.5 (PF0)
- net COL8: now also U3.45 (PB8); no longer U3.46 (PB9)
- net COL9: now also U3.43 (PB7), MX50.1; no longer MX48.1, U3.45 (PB8)
- net GND: now also J1.S1 (SHIELD), C?.2, R?.2
- net NRST: now also C?.1
- net ROW0: now also U3.38 (PA15); no longer U3.39 (PB3)
- net ROW2: now also U3.40 (PB4); no longer U3.41 (PB5)
- net ROW3: now also U3.39 (PB3); no longer U3.40 (PB4)
- net at D44.2 (A), MX44.2: now also MX50.2; no longer MX48.2
- net at D37.2 (A), MX37.2: now also MX48.2; no longer MX40.2
- net RGB MCU: now reaches U3.28 (PB15)
- net at D46.2 (A), MX46.2: now also MX51.2; no longer MX49.2
- net at D39.2 (A), MX39.2: now also MX49.2; no longer MX47.2
- net at D40.2 (A), MXsplit2.75.2: now also MXsplit2.25(1)1.2
- net at D36.2 (A), MX36.2, MXshift2.75.2: now also MX47.2
- net at D35.2 (A), MX35.2: now also MX40.2
- net at D47.2 (A), MXsplit2.25.2: now also MXsplit2.75(1)1.2
- no-connect marks 7 -> 2
Other:
- added sheet rgb (rgb.kicad_sch)
- note added: "NRST has internal pull up Hold high for normal operation"
- note added: "button to pull boot0 high while reseting to activate DFU"
- note removed: "JST"
- note removed: "Pico EZmate"
- moved on the sheet: S3
