File: Project/forti.kicad_sch (KiCad schematic)
At the start: 136 parts, among them J1 USB_C_Receptacle_USB2.0, U2 USBLC6-2SC6, U3 STM32F072C8Tx, U4 XC6206PxxxMR-Regulator_Linear

Commit message: new bottom row, proto project created, rgb revised
Parts:
- added MX52, MX55: MX_SW_HS, PCM_marbastlib-mx:SW_MX_1u, symbol PCM_marbastlib-mx:MX_SW_HS
- added MX53, MX54: MX_SW_HS, PCM_marbastlib-mx:SW_MX_1.5u, symbol PCM_marbastlib-mx:MX_SW_HS
Connections:
- net COL1: now also MX52.1
- net COL10: now also MX55.1
- net COL3: now also MX53.1
- net COL8: now also MX54.1
- net at D43.2 (A), MX43.2: now also MX54.2
- net at D45.2 (A), MX45.2: now also MX55.2
- net at D38.2 (A), MX38.2: now also MX52.2
- net at D41.2 (A), MX41.2: now also MX53.2
Other:
- moved on the sheet: S2, S3, S4, S5

Commit message: backup / cleanup
Parts:
- S1: value MX_stab -> 7
- S2, S4: value MX_stab -> 225
- S3, S5: value MX_stab -> 275
Other:
- moved on the sheet: S2, S4
Changed lines of the file:
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@@
   )
   (symbol (lib_id "PCM_marbastlib-mx:MX_SW_HS") (at 137.795 233.68 0) (unit 1)
-    (in_bom yes) (on_board yes) (dnp no) (fields_autoplaced)
-    (property "Reference" "MX53" (at 137.795 227.33 0)
+    (in_bom yes) (on_board yes) (dnp no)
+    (property "Reference" "MX53" (at 136.525 227.33 0)
       (effects (font (size 1.27 1.27)))
     )
@@
   )
   (symbol (lib_id "PCM_marbastlib-mx:MX_SW_HS") (at 82.55 233.68 0) (unit 1)
-    (in_bom yes) (on_board yes) (dnp no) (fields_autoplaced)
-    (property "Reference" "MX37" (at 82.55 227.33 0)
+    (in_bom yes) (on_board yes) (dnp no)
+    (property "Reference" "MX37" (at 82.55 229.87 0)
       (effects (font (size 1.27 1.27)))
     )
@@
     )
   )
-  (symbol (lib_id "PCM_marbastlib-mx:MX_stab") (at 143.51 252.095 0) (unit 1)
+  (symbol (lib_id "PCM_marbastlib-mx:MX_stab") (at 174.625 259.08 0) (unit 1)
     (in_bom yes) (on_board yes) (dnp no) (fields_autoplaced)
-    (property "Reference" "S2" (at 149.86 251.333 0)
+    (property "Reference" "S2" (at 180.975 258.318 0)
       (effects (font (size 1.27 1.27)) (justify left))
     )
-    (property "Value" "MX_stab" (at 149.86 253.873 0)
-      (effects (font (size 1.27 1.27)) (justify left) hide)
+    (property "Value" "225" (at 180.975 260.858 0)
+      (effects (font (size 1.27 1.27)) (justify left))
     )
-    (property "Footprint" "PCM_marbastlib-mx:STAB_MX_P_2.25u" (at 143.51 252.095 0)
+    (property "Footprint" "PCM_marbastlib-mx:STAB_MX_P_2.25u" (at 174.625 259.08 0)
       (effects (font (size 1.27 1.27)) hide)
     )
-    (property "Datasheet" "" (at 143.51 252.095 0)
+    (property "Datasheet" "" (at 174.625 259.08 0)
       (effects (font (size 1.27 1.27)) hide)
     )
@@
   )
   (symbol (lib_id "PCM_marbastlib-mx:MX_SW_HS") (at 107.95 233.68 0) (unit 1)
-    (in_bom yes) (on_board yes) (dnp no) (fields_autoplaced)
-    (property "Reference" "MX39" (at 107.95 227.33 0)
+    (in_bom yes) (on_board yes) (dnp no)
+    (property "Reference" "MX39" (at 107.95 229.87 0)
       (effects (font (size 1.27 1.27)))
     )
@@
       (effects (font (size 1.27 1.27)) (justify left))
     )
-    (property "Value" "MX_stab" (at 149.86 261.493 0)
-      (effects (font (size 1.27 1.27)) (justify left) hide)
+    (property "Value" "275" (at 149.86 261.493 0)
+      (effects (font (size 1.27 1.27)) (justify left))
     )
     (property "Footprint" "PCM_marbastlib-mx:STAB_MX_P_2.75u" (at 143.51 259.715 0)
@@
   )
   (symbol (lib_id "PCM_marbastlib-mx:MX_SW_HS") (at 208.915 233.68 0) (unit 1)
-    (in_bom yes) (on_board yes) (dnp no) (fields_autoplaced)
-    (property "Reference" "MX45" (at 208.915 227.965 0)
+    (in_bom yes) (on_board yes) (dnp no)
+    (property "Reference" "MX45" (at 208.915 229.87 0)
       (effects (font (size 1.27 1.27)))
     )
@@
   )
   (symbol (lib_id "PCM_marbastlib-mx:MX_SW_HS") (at 95.25 233.68 0) (unit 1)
-    (in_bom yes) (on_board yes) (dnp no) (fields_autoplaced)
-    (property "Reference" "MX38" (at 95.25 227.33 0)
+    (in_bom yes) (on_board yes) (dnp no)
+    (property "Reference" "MX38" (at 95.25 229.87 0)
       (effects (font (size 1.27 1.27)))
     )
@@
   (symbol (lib_id "PCM_marbastlib-mx:MX_SW_HS") (at 176.53 233.68 0) (unit 1)
     (in_bom yes) (on_board yes) (dnp no)
-    (property "Reference" "MXsplit2.75(1)1" (at 173.99 228.6 0)
+    (property "Reference" "MXsplit2.75(1)1" (at 171.45 228.6 0)
       (effects (font (size 1.27 1.27)))
     )
@@
     )
   )
-  (symbol (lib_id "PCM_marbastlib-mx:MX_stab") (at 174.625 259.715 0) (unit 1)
+  (symbol (lib_id "PCM_marbastlib-mx:MX_stab") (at 143.51 251.46 0) (unit 1)
     (in_bom yes) (on_board yes) (dnp no) (fields_autoplaced)
-    (property "Reference" "S4" (at 180.975 258.953 0)
+    (property "Reference" "S4" (at 149.86 250.698 0)
       (effects (font (size 1.27 1.27)) (justify left))
     )
-    (property "Value" "MX_stab" (at 180.975 261.493 0)
-      (effects (font (size 1.27 1.27)) (justify left) hide)
+    (property "Value" "225" (at 149.86 253.238 0)
+      (effects (font (size 1.27 1.27)) (justify left))
     )
-    (property "Footprint" "PCM_marbastlib-mx:STAB_MX_P_2.25u" (at 174.625 259.715 0)
+    (property "Footprint" "PCM_marbastlib-mx:STAB_MX_P_2.25u" (at 143.51 251.46 0)
       (effects (font (size 1.27 1.27)) hide)
     )
-    (property "Datasheet" "" (at 174.625 259.715 0)
+    (property "Datasheet" "" (at 143.51 251.46 0)
       (effects (font (size 1.27 1.27)) hide)
     )
@@
   )
   (symbol (lib_id "PCM_marbastlib-mx:MX_SW_HS") (at 133.35 233.68 0) (unit 1)
-    (in_bom yes) (on_board yes) (dnp no) (fields_autoplaced)
-    (property "Reference" "MX41" (at 133.35 227.33 0)
+    (in_bom yes) (on_board yes) (dnp no)
+    (property "Reference" "MX41" (at 133.35 229.87 0)
       (effects (font (size 1.27 1.27)))
     )
@@
       (effects (font (size 1.27 1.27)) (justify left))
     )
-    (property "Value" "MX_stab" (at 165.1 253.873 0)
-      (effects (font (size 1.27 1.27)) (justify left) hide)
+    (property "Value" "7" (at 165.1 253.873 0)
+      (effects (font (size 1.27 1.27)) (justify left))
     )
     (property "Footprint" "PCM_marbastlib-mx:STAB_MX_P_7u" (at 158.75 252.095 0)
@@
   )
   (symbol (lib_id "PCM_marbastlib-mx:MX_SW_HS") (at 221.615 233.68 0) (unit 1)
-    (in_bom yes) (on_board yes) (dnp no) (fields_autoplaced)
-    (property "Reference" "MX46" (at 221.615 227.965 0)
+    (in_bom yes) (on_board yes) (dnp no)
+    (property "Reference" "MX46" (at 221.615 229.87 0)
       (effects (font (size 1.27 1.27)))
     )
@@
   )
   (symbol (lib_id "PCM_marbastlib-mx:MX_SW_HS") (at 183.515 233.68 0) (unit 1)
-    (in_bom yes) (on_board yes) (dnp no) (fields_autoplaced)
-    (property "Reference" "MX43" (at 183.515 227.965 0)
+    (in_bom yes) (on_board yes) (dnp no)
+    (property "Reference" "MX43" (at 183.515 229.87 0)
       (effects (font (size 1.27 1.27)))
     )
@@
   (symbol (lib_id "PCM_marbastlib-mx:MX_SW_HS") (at 151.13 233.68 0) (unit 1)
     (in_bom yes) (on_board yes) (dnp no)
-    (property "Reference" "MXsplit2.25(1)1" (at 149.86 228.6 0)
+    (property "Reference" "MXsplit2.25(1)1" (at 147.32 228.6 0)
       (effects (font (size 1.27 1.27)))
     )
@@
       (effects (font (size 1.27 1.27)) (justify left))
     )
-    (property "Value" "MX_stab" (at 180.975 253.873 0)
-      (effects (font (size 1.27 1.27)) (justify left) hide)
+    (property "Value" "275" (at 180.975 253.873 0)
+      (effects (font (size 1.27 1.27)) (justify left))
     )
     (property "Footprint" "PCM_marbastlib-mx:STAB_MX_P_2.75u" (at 174.625 252.095 0)
@@
   )
   (symbol (lib_id "PCM_marbastlib-mx:MX_SW_HS") (at 196.215 233.68 0) (unit 1)
-    (in_bom yes) (on_board yes) (dnp no) (fields_autoplaced)
-    (property "Reference" "MX44" (at 196.215 227.965 0)
+    (in_bom yes) (on_board yes) (dnp no)
+    (property "Reference" "MX44" (at 196.215 229.87 0)
       (effects (font (size 1.27 1.27)))
     )
@@
   )
   (symbol (lib_id "PCM_marbastlib-mx:MX_SW_HS") (at 158.115 233.68 0) (unit 1)
-    (in_bom yes) (on_board yes) (dnp no) (fields_autoplaced)
-    (property "Reference" "MX42" (at 158.115 227.965 0)
+    (in_bom yes) (on_board yes) (dnp no)
+    (property "Reference" "MX42" (at 158.115 229.87 0)
       (effects (font (size 1.27 1.27)))
     )
@@
   (symbol (lib_id "PCM_marbastlib-mx:MX_SW_HS") (at 146.05 233.68 0) (unit 1)
     (in_bom yes) (on_board yes) (dnp no)
-    (property "Reference" "MXsplit2.75" (at 144.78 226.06 0)
+    (property "Reference" "MXsplit2.75" (at 146.05 226.06 0)
       (effects (font (size 1.27 1.27)))
     )

Commit message: two different pcb versions
Parts:
- removed C3: 4.7uF, Capacitor_SMD:C_0603_1608Metric, symbol Device:C_Small
- C16, C17: LCSC C52923 -> (none)
- C3: renamed from C4; value 1uF -> 10uF
- C?: LCSC C307331 -> (none)
- R3, R4: LCSC C25905 -> (none)
- renumbered C5 to C4, C6 to C5, C7 to C6, C8 to C7, C9 to C8, D41 to D40, D40 to D41, D47 to D43, D43 to D44, D44 to D45, D45 to D46, D46 to D47, MX40 to MX36, MX36 to MX37, MX47 to MX38, MX37 to MX39, MX48 to MX40, MX38 to MX41, MX52 to MX42, MX39 to MX43, MX49 to MX44, MX41 to MX45, MX53 to MX46, MX42 to MX47, MX43 to MX48, MX54 to MX49, MX44 to MX50, MX50 to MX51, MX45 to MX52, MX55 to MX53, MX46 to MX54, MX51 to MX55, MXenter2.25 to MXenter2.1, MXshift2.25 to MXshift2.1, MXshift2.75 to MXshift2.2, MXsplit2.75 to MXsplit2.1, MXsplit2.25 to MXsplit2.2, S4 to S1, S1 to S2, S5 to S3, S2 to S4, S3 to S5, U3 to U2, enter2.25 to enter2.1, shift2.75 to shift2.1, shift2.25 to shift2.2
