File: Project/forti rev 2.kicad_sch (KiCad schematic)
At the start: 139 parts, among them J1 USB_C_Receptacle_USB2.0, U2 STM32F072C8Tx, U2 USBLC6-2SC6, U4 XC6206PxxxMR-Regulator_Linear

Commit message: backup
Parts:
- S1, S4, shift2.2: footprint PCM_marbastlib-mx:STAB_MX_P_2.25u -> PCM_marbastlib-mx:STAB_MX_2.25u
- S2: footprint PCM_marbastlib-mx:STAB_MX_P_7u -> PCM_marbastlib-mx:STAB_MX_7u
- S3, S5, shift2.1: footprint PCM_marbastlib-mx:STAB_MX_P_2.75u -> PCM_marbastlib-mx:STAB_MX_2.75u
