File: Project/forti rev 3.kicad_pcb (KiCad board)
At the start: 2 copper layers, 245.7 x 82.9 mm, 164 parts, among them J1 USB_C_Receptacle_USB2.0, SW1 SKQGABE010, U1 USBLC6-2SC6, U2 STM32F072C8Tx, U3 XC6206PxxxMR-Regulator_Linear, U4 74AHCT1G125

Commit message: revision
usb needs fix still
Parts:
- removed C10: 100nF, Capacitor_SMD:C_0603_1608Metric
- removed the G*** at (108.0, 97.6)
- removed the G*** at (193.7, 97.6)
- removed the G*** at (195.3, 96.0)
- removed the G*** at (104.8, 96.0)
- removed the G*** at (44.2, 47.5)
- removed LED1, LED10, LED11, LED12, LED13, LED14, LED15, LED16, LED17, LED18, LED2, LED3, LED4, LED5, LED6, LED7, LED8, LED9: WS2812_2020, PCM_marbastlib-various:LED_WS2812_2020
- removed U4: 74AHCT1G125, Package_TO_SOT_SMD:TSOT-23-5
- added G***: LOGO, LOGO, F.Cu at (108.0, 98.4)
- added G***: LOGO, LOGO, F.Cu at (193.7, 98.4)
- added G***: LOGO, LOGO, B.Cu at (104.8, 97.6)
- added G***: LOGO, LOGO, B.Cu at (44.2, 47.5)
- added G***: LOGO, LOGO, B.Cu at (195.3, 97.6)
- S1, S4, enter2.1, shift2.2: footprint PCM_marbastlib-mx:STAB_MX_P_2.25u -> PCM_marbastlib-mx:STAB_MX_2.25u
- S2: footprint PCM_marbastlib-mx:STAB_MX_P_7u -> PCM_marbastlib-mx:STAB_MX_7u
- S3, S5, shift2.1: footprint PCM_marbastlib-mx:STAB_MX_P_2.75u -> PCM_marbastlib-mx:STAB_MX_2.75u
- moved R1 2.98 mm to (244.5, 33.5), turned to 0 degrees
Routing:
- net +5V: track 833.6 -> 185.5 mm, vias 21 -> 0
- net GND: track 932.7 -> 511.5 mm, vias 35 -> 15
- net rgb underglow: track 60.2 -> 0.00 mm
- net Net-(LED13-DOUT): track 44.0 -> 0.00 mm, vias 2 -> 0
- net Net-(LED14-DOUT): track 20.2 -> 0.00 mm
- net Net-(LED17-DOUT): track 20.0 -> 0.00 mm, vias 2 -> 0
- net Net-(LED5-DOUT): track 20.0 -> 0.00 mm
- net Net-(LED4-DOUT): track 19.3 -> 0.00 mm
- net Net-(LED10-DOUT): track 18.1 -> 0.00 mm
- net Net-(LED10-DIN): track 17.8 -> 0.00 mm
- net Net-(LED8-DOUT): track 17.7 -> 0.00 mm
- net Net-(LED16-DOUT): track 17.7 -> 0.00 mm, vias 2 -> 0
- net Net-(LED2-DOUT): track 17.6 -> 0.00 mm
- net Net-(LED1-DOUT): track 17.6 -> 0.00 mm
- net Net-(LED7-DOUT): track 17.6 -> 0.00 mm
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Other:
- board text added: "MOVE By 1mm"
- board text added: "boot"
- board text added: "step"
- board text removed: "stepped"

Commit message: update production files v3
Routing:
- net GND: track 511.5 -> 527.8 mm
- net COL1: track 96.4 -> 97.4 mm
- net Net-(D3-A): track 3.05 -> 3.57 mm
- net Net-(D2-A): track 3.05 -> 3.57 mm
Other:
- board text removed: "MOVE By 1mm"
