File: Project/Other PCB versions/EC-wip/EC matrix.kicad_sch (KiCad schematic)
At the start: 55 parts

Commit message: EC progress
Parts:
- removed SW_EC55, SW_EC58: 1.5u, cipulot_parts:ecs_pad_1U_no_ring, symbol cipulot_parts:Topre
- SW_EC1, SW_EC10, SW_EC11, SW_EC12, SW_EC13, SW_EC14, SW_EC15, SW_EC16, SW_EC17, SW_EC18, SW_EC19, SW_EC2, SW_EC20, SW_EC21, SW_EC22, SW_EC23, SW_EC24, SW_EC25, SW_EC26, SW_EC27, SW_EC28, SW_EC29, SW_EC3, SW_EC30, SW_EC31, SW_EC32, SW_EC33, SW_EC34, SW_EC37, SW_EC4, SW_EC40, SW_EC41, SW_EC42, SW_EC43, SW_EC44, SW_EC46, SW_EC47, SW_EC48, SW_EC49, SW_EC5, SW_EC50, SW_EC52, SW_EC6, SW_EC7, SW_EC8, SW_EC9: symbol cipulot_parts:Topre -> cipulot_parts:EC_SW
- SW_EC35, SW_EC36: symbol cipulot_parts:Topre -> cipulot_parts:EC_SW_1u&1.75u
- SW_EC38, SW_EC60, SW_EC61: footprint cipulot_parts:ecs_pad_1U_no_ring -> cipulot_parts:ecs_pad_1U_no_ring_1u_edge_cut; symbol cipulot_parts:Topre -> cipulot_parts:EC_SW
- SW_EC39, SW_EC45: footprint cipulot_parts:ecs_pad_1U_no_ring -> cipulot_parts:ecs_pad_no_ring_stepped&normal_cut; symbol cipulot_parts:Topre -> cipulot_parts:EC_SW
Connections:
- net COL0: now also SW_EC1.1, SW_EC13.1, SW_EC25.1, SW_EC37.1, SW_EC50.1; no longer SW_EC1.2, SW_EC13.2, SW_EC25.2, SW_EC37.2, SW_EC50.2
- net COL1: now also SW_EC14.1, SW_EC2.1, SW_EC26.1, SW_EC38.1, SW_EC61.1; no longer SW_EC14.2, SW_EC2.2, SW_EC26.2, SW_EC38.2, SW_EC61.2
- net COL10: now also SW_EC11.1, SW_EC23.1, SW_EC46.1, SW_EC60.2; no longer SW_EC11.2, SW_EC23.2, SW_EC47.2
- net COL11: now also SW_EC12.1, SW_EC24.1, SW_EC47.1, SW_EC48.1, SW_EC49.1; no longer SW_EC12.2, SW_EC24.2, SW_EC48.2, SW_EC49.2
- net COL2: now also SW_EC15.1, SW_EC27.1, SW_EC3.1, SW_EC39.1; no longer SW_EC15.2, SW_EC27.2, SW_EC3.2, SW_EC39.2
- net COL3: now also SW_EC16.1, SW_EC28.1, SW_EC4.1, SW_EC40.1; no longer SW_EC16.2, SW_EC28.2, SW_EC4.2, SW_EC40.2
- net COL4: now also SW_EC17.1, SW_EC29.1, SW_EC41.1, SW_EC5.1; no longer SW_EC17.2, SW_EC29.2, SW_EC41.2, SW_EC5.2
- net COL5: now also SW_EC18.1, SW_EC30.1, SW_EC6.1; no longer SW_EC18.2, SW_EC30.2, SW_EC42.2, SW_EC6.2
- net COL6: now also SW_EC19.1, SW_EC31.1, SW_EC42.1, SW_EC7.1; no longer SW_EC19.2, SW_EC31.2, SW_EC43.2, SW_EC7.2
- net COL7: now also SW_EC20.1, SW_EC32.1, SW_EC43.1, SW_EC8.1; no longer SW_EC20.2, SW_EC32.2, SW_EC44.2, SW_EC8.2
- net COL8: now also SW_EC21.1, SW_EC33.1, SW_EC44.1, SW_EC9.1; no longer SW_EC21.2, SW_EC33.2, SW_EC45.2, SW_EC9.2
- net COL9: now also SW_EC10.1, SW_EC22.1, SW_EC34.1, SW_EC45.2; no longer SW_EC10.2, SW_EC22.2, SW_EC34.2, SW_EC46.2, SW_EC60.2
- net GND: now also SW_EC35.4 (SG), SW_EC36.4 (SG); no longer SW_EC35.3, SW_EC36.3
- net ROW0: now also SW_EC1.2, SW_EC10.2, SW_EC11.2, SW_EC12.2, SW_EC2.2, SW_EC3.2, SW_EC4.2, SW_EC5.2, SW_EC6.2, SW_EC7.2, SW_EC8.2, SW_EC9.2; no longer SW_EC1.1, SW_EC10.1, SW_EC11.1, SW_EC12.1, SW_EC2.1, SW_EC3.1, SW_EC4.1, SW_EC5.1, SW_EC6.1, SW_EC7.1, SW_EC8.1, SW_EC9.1
- net ROW1: now also SW_EC13.2, SW_EC14.2, SW_EC15.2, SW_EC16.2, SW_EC17.2, SW_EC18.2, SW_EC19.2, SW_EC20.2, SW_EC21.2, SW_EC22.2, SW_EC23.2, SW_EC24.2, SW_EC48.2, SW_EC49.2; no longer SW_EC13.1, SW_EC14.1, SW_EC15.1, SW_EC16.1, SW_EC17.1, SW_EC18.1, SW_EC19.1, SW_EC20.1, SW_EC21.1, SW_EC22.1, SW_EC23.1, SW_EC24.1, SW_EC48.1, SW_EC49.1
- net ROW2: now also SW_EC25.2, SW_EC26.2, SW_EC27.2, SW_EC28.2, SW_EC29.2, SW_EC30.2, SW_EC31.2, SW_EC32.2, SW_EC33.2, SW_EC34.2, SW_EC35.3, SW_EC36.3, SW_EC50.2; no longer SW_EC25.1, SW_EC26.1, SW_EC27.1, SW_EC28.1, SW_EC29.1, SW_EC30.1, SW_EC31.1, SW_EC32.1, SW_EC33.1, SW_EC34.1, SW_EC50.1
- net ROW3: now also SW_EC37.2, SW_EC38.2, SW_EC39.2, SW_EC40.2, SW_EC41.2, SW_EC42.2, SW_EC43.2, SW_EC44.2, SW_EC46.2, SW_EC47.2, SW_EC61.2; no longer SW_EC37.1, SW_EC38.1, SW_EC39.1, SW_EC40.1, SW_EC41.1, SW_EC42.1, SW_EC43.1, SW_EC44.1, SW_EC46.1, SW_EC47.1, SW_EC61.1
Other:
- note added: "MOVE BY ONE COL"
- note added: "RIGHT WIRING?"
- moved on the sheet: SW_EC1, SW_EC10, SW_EC11, SW_EC12, SW_EC13, SW_EC15, SW_EC16, SW_EC17, SW_EC18, SW_EC19, SW_EC2, SW_EC20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

Commit message: progress on EC version
Parts:
- SW_EC23, SW_EC49: footprint cipulot_parts:ecs_pad_1U_no_ring -> cipulot_parts:ecs_pad_1U_no_ring_1u_edge_cut
Connections:
- net COL10: now also SW_EC23.2; no longer SW_EC23.1, SW_EC52.2
- net COL11: now also SW_EC36.1, SW_EC36.3, SW_EC52.2; no longer SW_EC36.2
- net ROW1: now also SW_EC23.1; no longer SW_EC23.2
- net ROW2: now also SW_EC36.2; no longer SW_EC36.1, SW_EC36.3

Commit message: EC bottom row and mounting holes
need to double check routing 90°
Parts:
- removed SW_EC60, SW_EC61: 1u, cipulot_parts:ecs_pad_1U_no_ring_1u_edge_cut, symbol cipulot_parts:EC_SW
- SW_EC37, SW_EC40, SW_EC44, SW_EC47: value stepped -> 1u; footprint cipulot_parts:ecs_pad_no_ring_stepped&normal -> cipulot_parts:ecs_pad_1U_no_ring
- SW_EC38: footprint cipulot_parts:ecs_pad_1U_no_ring_1u_edge_cut -> cipulot_parts:ecs_pad_1U_no_ring
- SW_EC39, SW_EC45: value 1u -> stepped
- SW_EC41, SW_EC43: value Topre -> split
- SW_EC42: value Topre -> 6u 7u
Connections:
- net COL2: now also SW_EC39.2; no longer SW_EC39.1
- net ROW3: now also SW_EC39.1; no longer SW_EC39.2
