File: Project/Other PCB versions/EC-wip/forti EC.kicad_pcb (KiCad board)
At the start: 4 copper layers, 245.7 x 83.6 mm, 153 parts, among them J2 USB_C_Receptacle_USB2.0, SW1 BOOT0, U1 USBLC6-2SC6, U2 XC6206PxxxMR-Regulator_Linear, U3 OPA354, U4 74AHCT1G125, U5 74HC4051, U7 74HC4051, U8 STM32F401CBUx, Y1 8 MHz

Commit message: EC bottom row and mounting holes
need to double check routing 90°
Parts:
- removed SW_EC60, SW_EC61: 1u, cipulot_parts:ecs_pad_1U_no_ring_1u_edge_cut
- SW_EC37, SW_EC40, SW_EC44, SW_EC47: value stepped -> 1u; footprint cipulot_parts:ecs_pad_no_ring_stepped&normal -> cipulot_parts:ecs_pad_1U_no_ring
- SW_EC38: footprint cipulot_parts:ecs_pad_1U_no_ring_1u_edge_cut -> cipulot_parts:ecs_pad_1U_no_ring
- SW_EC39, SW_EC45: value 1u -> stepped
- SW_EC41, SW_EC43: value Topre -> split
- SW_EC42: value Topre -> 6u 7u
- moved H24 193.8 mm to (-3.15, 73.8)
- moved H25 193.8 mm to (-3.15, 77.0)
- moved H26 193.8 mm to (-3.15, 80.2)
- moved H16 136.7 mm to (45.2, 98.4)
- moved H20 122.1 mm to (64.3, 98.4)
- moved H15 88.8 mm to (207.2, 41.3)
- moved H18 84.5 mm to (102.4, 98.4)
- moved H17 83.2 mm to (254.8, 98.4)
- moved H14 79.8 mm to (221.5, 79.4)
- moved H22 79.7 mm to (135.7, 60.3)
- moved H21 73.4 mm to (235.7, 98.4)
- moved H19 44.0 mm to (197.6, 98.4)
- moved H4 38.1 mm to (169.1, 41.3)
- moved H23 37.4 mm to (159.5, 98.4)
- moved H13 23.8 mm to (185.7, 98.4)
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Connections:
- SW_EC39 pad 1: COL2 -> ROW3
- SW_EC39 pad 2: ROW3 -> COL2
Routing:
- net ROW3: track 453.0 -> 430.3 mm, vias 22 -> 16
- net COL1: track 130.7 -> 122.3 mm, vias 5 -> 4
- net AMUX_SEL_1: track 235.1 -> 241.2 mm
- net AMUX_SEL_0: track 235.4 -> 241.0 mm
- net COL3: track 86.7 -> 81.2 mm, vias 5 -> 4
- net COL10: track 152.5 -> 147.0 mm, vias 6 -> 5
- net COL9: track 117.9 -> 112.8 mm
- net COL8: track 92.1 -> 87.4 mm, vias 5 -> 4
- net AMUX_SEL_2: track 235.1 -> 239.5 mm
- net COL2: track 111.2 -> 106.8 mm
- net COL0: track 187.2 -> 184.0 mm, vias 7 -> 6
- net COL4: track 87.0 -> 84.7 mm
- net APLEX_EN_PIN_0: track 91.9 -> 89.9 mm
- net VBAT: track 254.1 -> 252.6 mm
- net COL7: track 80.5 -> 81.8 mm
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Other:
- board text added: "7 6"
- board text added: "make sure 90s crossings are there"
- board text removed: "7"
- board text removed: "EDIT BOTTOMROW, MOUNTING HOLES"

Commit message: forti work
Parts:
- moved LED17 3.17 mm to (270.7, 50.8)
Routing:
- net Net-(LED16-DIN): track 22.2 -> 19.1 mm
- net Net-(LED17-DIN): track 14.0 -> 17.2 mm
