File: Project/Other PCB versions/EC-wip/forti EC.kicad_sch (KiCad schematic)
At the start: 27 parts, among them J1 USB_C_Receptacle_USB2.0, SW38 BOOT0, U1 STM32F401CBUx, U2 USBLC6-2SC6, U4 XC6206PxxxMR-Regulator_Linear, Y1 8 MHz

Commit message: EC progress
Connections:
- net ADC: now also U1.43 (PB7); no longer U1.13 (PA3)
- net AMUX_SEL_0: now also U1.39 (PB3); no longer U1.41 (PB5)
- net AMUX_SEL_1: now also U1.38 (PA15); no longer U1.40 (PB4)
- net AMUX_SEL_2: now also U1.37 (PA14); no longer U1.39 (PB3)
- net APLEX_EN_PIN_0: now also U1.41 (PB5); no longer U1.18 (PB0)
- net APLEX_EN_PIN_1: now also U1.40 (PB4); no longer U1.19 (PB1)
- net DISCHARGE_PIN: now also U1.42 (PB6); no longer U1.14 (PA4)
- net RGB MCU: now also U1.12 (PA2)
- net ROW0: now also R2.1; no longer R9.2
- net ROW1: now also R1.2; no longer R8.1
- net ROW2: now also R9.2; no longer R2.1
- net ROW3: now also R8.1; no longer R1.2
- net SWCLK: no longer U1.37 (PA14)
- net SWDIO: no longer U1.34 (PA13)
- net at U1.15 (PA5): now also R8.2
- net at U1.16 (PA6): now also R2.2
- net at R1.1: now also U1.13 (PA3); no longer U1.25 (PB12)
- net at R9.1: now also U1.14 (PA4); no longer U1.26 (PB13)
- net at U1.27 (PB14): no longer R8.2
- net at U1.28 (PB15): no longer R2.2
- no-connect marks 19 -> 5
Other:
- moved on the sheet: R1, R2, R8, R9

Commit message: two different pcb versions
Changed lines of the file:
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@@
-    )
-  )
-  (global_label "SWCLK" (shape input) (at 25.4 109.22 0) (fields_autoplaced)
-    (effects (font (size 1.27 1.27)) (justify left))
-    (property "Intersheetrefs" "${INTERSHEET_REFS}" (at 34.0421 109.2994 0)
-      (effects (font (size 1.27 1.27)) (justify left) hide)
     )
   )
@@
     )
   )
-  (global_label "COL6" (shape input) (at 5.08 72.39 180) (fields_autoplaced)
-    (effects (font (size 1.27 1.27)) (justify right))
-    (property "Intersheetrefs" "${INTERSHEET_REFS}" (at -2.6639 72.39 0)
-      (effects (font (size 1.27 1.27)) (justify right) hide)
-    )
-  )
-  (global_label "ROW3" (shape input) (at 5.08 90.17 180) (fields_autoplaced)
-    (effects (font (size 1.27 1.27)) (justify right))
-    (property "Intersheetrefs" "${INTERSHEET_REFS}" (at -3.0872 90.17 0)
-      (effects (font (size 1.27 1.27)) (justify right) hide)
-    )
-  )
-  (global_label "ROW0" (shape input) (at 5.08 85.09 180) (fields_autoplaced)
-    (effects (font (size 1.27 1.27)) (justify right))
-    (property "Intersheetrefs" "${INTERSHEET_REFS}" (at -3.0872 85.09 0)
-      (effects (font (size 1.27 1.27)) (justify right) hide)
-    )
-  )
-  (global_label "COL2" (shape input) (at 5.08 67.31 180) (fields_autoplaced)
-    (effects (font (size 1.27 1.27)) (justify right))
-    (property "Intersheetrefs" "${INTERSHEET_REFS}" (at -2.6639 67.31 0)
-      (effects (font (size 1.27 1.27)) (justify right) hide)
-    )
-  )
   (global_label "XTAL1" (shape input) (at 57.15 53.34 180) (fields_autoplaced)
     (effects (font (size 1.27 1.27)) (justify right))
@@
     (effects (font (size 1.27 1.27)) (justify right))
     (property "Intersheetrefs" "${INTERSHEET_REFS}" (at 48.6288 73.5806 0)
-      (effects (font (size 1.27 1.27)) (justify right) hide)
-    )
-  )
-  (global_label "COL7" (shape input) (at 5.08 105.41 180) (fields_autoplaced)
-    (effects (font (size 1.27 1.27)) (justify right))
-    (property "Intersheetrefs" "${INTERSHEET_REFS}" (at -2.6639 105.41 0)
       (effects (font (size 1.27 1.27)) (justify right) hide)
     )
@@
     )
   )
-  (global_label "COL0" (shape input) (at 5.08 110.49 180) (fields_autoplaced)
-    (effects (font (size 1.27 1.27)) (justify right))
-    (property "Intersheetrefs" "${INTERSHEET_REFS}" (at -2.6639 110.49 0)
-      (effects (font (size 1.27 1.27)) (justify right) hide)
-    )
-  )
   (global_label "AMUX_SEL_1" (shape output) (at 90.17 104.14 0) (fields_autoplaced)
     (effects (font (size 1.27 1.27)) (justify left))
     (property "Intersheetrefs" "${INTERSHEET_REFS}" (at 104.6871 104.14 0)
-      (effects (font (size 1.27 1.27)) (justify left) hide)
-    )
-  )
-  (global_label "COL8" (shape input) (at 5.08 102.87 180) (fields_autoplaced)
-    (effects (font (size 1.27 1.27)) (justify right))
-    (property "Intersheetrefs" "${INTERSHEET_REFS}" (at -2.6639 102.87 0)
-      (effects (font (size 1.27 1.27)) (justify right) hide)
-    )
-  )
-  (global_label "SWDIO" (shape input) (at 25.4 106.68 0) (fields_autoplaced)
-    (effects (font (size 1.27 1.27)) (justify left))
-    (property "Intersheetrefs" "${INTERSHEET_REFS}" (at 33.6793 106.7594 0)
       (effects (font (size 1.27 1.27)) (justify left) hide)
     )
@@
     )
   )
-  (global_label "ROW1" (shape input) (at 5.08 87.63 180) (fields_autoplaced)
-    (effects (font (size 1.27 1.27)) (justify right))
-    (property "Intersheetrefs" "${INTERSHEET_REFS}" (at -3.0872 87.63 0)
-      (effects (font (size 1.27 1.27)) (justify right) hide)
-    )
-  )
   (global_label "VDD3" (shape input) (at 77.47 27.94 90) (fields_autoplaced)
     (effects (font (size 1.27 1.27)) (justify left))
@@
     (property "Intersheetrefs" "${INTERSHEET_REFS}" (at 74.8506 20.6888 90)
       (effects (font (size 1.27 1.27)) (justify left) hide)
-    )
-  )
-  (global_label "COL11" (shape input) (at 5.08 95.25 180) (fields_autoplaced)
-    (effects (font (size 1.27 1.27)) (justify right))
-    (property "Intersheetrefs" "${INTERSHEET_REFS}" (at -3.8734 95.25 0)
-      (effects (font (size 1.27 1.27)) (justify right) hide)
     )
   )
@@
     )
   )
-  (global_label "COL9" (shape input) (at 5.08 100.33 180) (fields_autoplaced)
-    (effects (font (size 1.27 1.27)) (justify right))
-    (property "Intersheetrefs" "${INTERSHEET_REFS}" (at -2.6639 100.33 0)
-      (effects (font (size 1.27 1.27)) (justify right) hide)
-    )
-  )
-  (global_label "COL3" (shape input) (at 5.08 64.77 180) (fields_autoplaced)
-    (effects (font (size 1.27 1.27)) (justify right))
-    (property "Intersheetrefs" "${INTERSHEET_REFS}" (at -2.6639 64.77 0)
-      (effects (font (size 1.27 1.27)) (justify right) hide)
-    )
-  )
   (global_label "VBAT" (shape input) (at 69.85 27.94 90) (fields_autoplaced)
     (effects (font (size 1.27 1.27)) (justify left))
     (property "Intersheetrefs" "${INTERSHEET_REFS}" (at 69.7706 21.1121 90)
       (effects (font (size 1.27 1.27)) (justify left) hide)
-    )
-  )
-  (global_label "COL1" (shape input) (at 5.08 107.95 180) (fields_autoplaced)
-    (effects (font (size 1.27 1.27)) (justify right))
-    (property "Intersheetrefs" "${INTERSHEET_REFS}" (at -2.6639 107.95 0)
-      (effects (font (size 1.27 1.27)) (justify right) hide)
     )
   )
@@
       (effects (font (size 1.27 1.27)) (justify right) hide)
     )
-  )
-  (global_label "COL10" (shape input) (at 5.08 97.79 180) (fields_autoplaced)
-    (effects (font (size 1.27 1.27)) (justify right))
-    (property "Intersheetrefs" "${INTERSHEET_REFS}" (at -3.8734 97.79 0)
-      (effects (font (size 1.27 1.27)) (justify right) hide)
-    )
-  )
-  (global_label "COL5" (shape input) (at 5.08 74.93 180) (fields_autoplaced)
-    (effects (font (size 1.27 1.27)) (justify right))
-    (property "Intersheetrefs" "${INTERSHEET_REFS}" (at -2.6639 74.93 0)
-      (effects (font (size 1.27 1.27)) (justify right) hide)
-    )
-  )
-  (global_label "COL4" (shape input) (at 5.08 77.47 180) (fields_autoplaced)
-    (effects (font (size 1.27 1.27)) (justify right))
-    (property "Intersheetrefs" "${INTERSHEET_REFS}" (at -2.6639 77.47 0)
-      (effects (font (size 1.27 1.27)) (justify right) hide)
-    )
-  )
-  (global_label "ROW2" (shape input) (at 5.08 92.71 180) (fields_autoplaced)
-    (effects (font (size 1.27 1.27)) (justify right))
-    (property "Intersheetrefs" "${INTERSHEET_REFS}" (at -3.0872 92.71 0)
-      (effects (font (size 1.27 1.27)) (justify right) hide)
-    )
