File: Project/EC-wip/forti EC.kicad_sch (KiCad schematic)
At the start: 27 parts, among them J1 USB_C_Receptacle_USB2.0, SW38 BOOT0, U1 STM32F401CBUx, U2 USBLC6-2SC6, U4 XC6206PxxxMR-Regulator_Linear, Y1 8 MHz

Commit message: update production files v3
Other:
- removed sheet rgb
- moved on the sheet: C10, C11, C16, C17, C6, C7, C8, C9, D_PWR1, F1, J1, R3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
