File: Project/EC-wip/forti EC.kicad_pcb (KiCad board)
At the start: 4 copper layers, 245.7 x 82.9 mm, 129 parts, among them J2 USB_C_Receptacle_USB2.0, SW1 BOOT0, U1 USBLC6-2SC6, U2 XC6206PxxxMR-Regulator_Linear, U3 OPA354, U5 74HC4051, U7 74HC4051, U8 STM32F401CBUx, Y1 8 MHz

Commit message: rev 4
Parts:
- added G***: LOGO, LOGO, F.Cu at (246.9, 49.2)
- moved G*** 0.83 mm to (245.7, 48.5)
Changed lines of the file:
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@@
 		)
 	)
+	(footprint "LOGO"
+		(layer "F.Cu")
+		(at 246.85625 49.2125)
+		(property "Reference" "G***"
+			(at 0 0 0)
+			(layer "F.SilkS")
+			(hide yes)
+			(effects
+				(font
+					(size 1.5 1.5)
+					(thickness 0.3)
+				)
+			)
+		)
+		(property "Value" "LOGO"
+			(at 0.75 0 0)
+			(layer "F.SilkS")
+			(hide yes)
+			(effects
+				(font
+					(size 1.5 1.5)
+					(thickness 0.3)
+				)
+			)
+		)
+		(property "Footprint" ""
+			(at 0 0 0)
+			(layer "F.Fab")
+			(hide yes)
+			(effects
+				(font
+					(size 1.27 1.27)
+					(thickness 0.15)
+				)
+			)
+		)
+		(property "Datasheet" ""
+			(at 0 0 0)
+			(layer "F.Fab")
+			(hide yes)
+			(effects
+				(font
+					(size 1.27 1.27)
+					(thickness 0.15)
+				)
+			)
+		)
+		(property "Description" ""
+			(at 0 0 0)
+			(layer "F.Fab")
+			(hide yes)
+			(effects
+				(font
+					(size 1.27 1.27)
+					(thickness 0.15)
+				)
+			)
+		)
+		(attr board_only exclude_from_pos_files exclude_from_bom)
+		(fp_poly
+			(pts
+				(xy 1.52723 -0.066505) (xy 1.797967 0.204264) (xy 1.429817 0.204264) (xy 1.061667 0.204264) (xy 0.790929 -0.066505)
+				(xy 0.520192 -0.337273) (xy 0.888342 -0.337273) (xy 1.256493 -0.337273)
+			)
+			(stroke
+				(width 0)
+				(type solid)
+			)
+			(fill solid)
+			(layer "F.SilkS")
+		)
+		(fp_poly
+			(pts
+				(xy 0.592611 0.200709) (xy 0.652193 0.260315) (xy 0.709926 0.318113) (xy 0.765453 0.373746) (xy 0.818419 0.426854)
+				(xy 0.868469 0.477081) (xy 0.915245 0.524068) (xy 0.958394 0.567456) (xy 0.997558 0.606888) (xy 1.032382 0.642006)
+				(xy 1.062511 0.672452) (xy 1.087588 0.697867) (xy 1.107259 0.717894) (xy 1.121167 0.732173) (xy 1.128956 0.740348)
+				(xy 1.130578 0.742246) (xy 1.125948 0.742811) (xy 1.112544 0.743348) (xy 1.091092 0.74385) (xy 1.062316 0.744311)
+				(xy 1.026943 0.744723) (xy 0.9857 0.745078) (xy 0.939311 0.745371) (xy 0.888504 0.745593) (xy 0.834003 0.745739)
+				(xy 0.776535 0.7458) (xy 0.765982 0.745801) (xy 0.401387 0.745801) (xy -0.140135 0.204264) (xy -0.681657 -0.337273)
+				(xy -0.313506 -0.337273) (xy 0.054644 -0.337273)
+			)
+			(stroke
+				(width 0)
+				(type solid)
+			)
+			(fill solid)
+			(layer "F.SilkS")
+		)
+		(fp_poly
+			(pts
+				(xy 1.201642 -2.315975) (xy 1.243781 -2.273782) (xy 1.283879 -2.233536) (xy 1.321441 -2.19574) (xy 1.355972 -2.160896)
+				(xy 1.386979 -2.129506) (xy 1.413965 -2.102073) (xy 1.436436 -2.079099) (xy 1.453897 -2.061086)
+				(xy 1.465853 -2.048538) (xy 1.47181 -2.041957) (xy 1.472396 -2.041066) (xy 1.467989 -2.037642) (xy 1.457453 -2.029643)
+				(xy 1.442263 -2.018185) (xy 1.423897 -2.004387) (xy 1.419628 -2.001186) (xy 1.300644 -1.917846)
+				(xy 1.175468 -1.841456) (xy 1.04471 -1.772336) (xy 0.908985 -1.710808) (xy 0.768904 -1.657191) (xy 0.749722 -1.650586)
+				(xy 0.712972 -1.638535) (xy 0.671451 -1.625651) (xy 0.627675 -1.612658) (xy 0.584159 -1.600279)
+				(xy 0.543419 -1.589239) (xy 0.50797 -1.580262) (xy 0.494034 -1.577002) (xy 0.478968 -1.573366) (xy 0.467742 -1.570225)
+				(xy 0.463859 -1.568777) (xy 0.466772 -1.566894) (xy 0.477456 -1.563221) (xy 0.49445 -1.5582) (xy 0.51629 -1.552274)
+				(xy 0.530364 -1.548657) (xy 0.679009 -1.50702) (xy 0.821309 -1.45858) (xy 0.957832 -1.40305) (xy 1.089147 -1.340146)
+				(xy 1.215822 -1.26958) (xy 1.338424 -1.191067) (xy 1.457522 -1.104322) (xy 1.53198 -1.044508) (xy 1.551617 -1.027508)
+				(xy 1.574806 -1.006371) (xy 1.600744 -0.98192) (xy 1.628632 -0.954979) (xy 1.657667 -0.926372) (xy 1.687048 -0.896921)
+				(xy 1.715973 -0.86745) (xy 1.743642 -0.838782) (xy 1.769252 -0.81174) (xy 1.792002 -0.787148) (xy 1.811091 -0.76583)
+				(xy 1.825717 -0.748607) (xy 1.83508 -0.736305) (xy 1.838376 -0.729747) (xy 1.833688 -0.729504) (xy 1.819872 -0.729267)
+				(xy 1.797299 -0.729036) (xy 1.766343 -0.728811) (xy 1.727375 -0.728595) (xy 1.680769 -0.728386)
+				(xy 1.626896 -0.728187) (xy 1.566128 -0.727998) (xy 1.498839 -0.72782) (xy 1.4254 -0.727653) (xy 1.346183 -0.727499)
+				(xy 1.261562 -0.727358) (xy 1.171908 -0.727231) (xy 1.077594 -0.727119) (xy 0.978992 -0.727022)
+				(xy 0.876474 -0.726942) (xy 0.770413 -0.726879) (xy 0.661181 -0.726834) (xy 0.549151 -0.726807)
+				(xy 0.452459 -0.7268) (xy -0.933458 -0.7268) (xy -1.398972 -0.261268) (xy -1.864485 0.204264) (xy -1.398972 0.669796)
+				(xy -0.933458 1.135328) (xy 0.928675 1.135328) (xy 2.790808 1.135328) (xy 1.859753 2.066392) (xy 0.928698 2.997456)
+				(xy -0.237517 2.997456) (xy -1.403731 2.997456) (xy -2.333603 2.067575) (xy -3.263475 1.137694)
+				(xy -3.263475 0.204255) (xy -3.263475 -0.729185) (xy -2.333594 -1.659057) (xy -1.403713 -2.588929)
+				(xy -0.237497 -2.588929) (xy 0.92872 -2.588929)
+			)
+			(stroke
+				(width 0)
+				(type solid)
+			)
+			(fill solid)
+			(layer "F.SilkS")
+		)
+		(fp_poly
+			(pts
+				(xy 2.5853 -3.075102) (xy 2.588193 -3.068708) (xy 2.592291 -3.055394) (xy 2.597987 -3.034186) (xy 2.600762 -3.023428)
+				(xy 2.639731 -2.890222) (xy 2.687407 -2.760683) (xy 2.743632 -2.635121) (xy 2.808249 -2.513845)
+				(xy 2.881102 -2.397164) (xy 2.962034 -2.285387) (xy 2.998411 -2.239959) (xy 3.042938 -2.188595)
+				(xy 3.093685 -2.134618) (xy 3.148576 -2.080041) (xy 3.205533 -2.026873) (xy 3.262479 -1.977128)
+				(xy 3.308603 -1.9396) (xy 3.408202 -1.867067) (xy 3.514456 -1.799975) (xy 3.625883 -1.739049) (xy 3.741 -1.685017)
+				(xy 3.858328 -1.638606) (xy 3.976382 -1.600542) (xy 4.028455 -1.586555) (xy 4.051415 -1.580734)
+				(xy 4.071402 -1.57559) (xy 4.086406 -1.571645) (xy 4.094419 -1.569422) (xy 4.094782 -1.569307) (xy 4.092942 -1.567414)
+				(xy 4.083243 -1.563708) (xy 4.067052 -1.55863) (xy 4.045739 -1.552621) (xy 4.030652 -1.548646) (xy 3.900005 -1.510243)
+				(xy 3.773259 -1.463347) (xy 3.650748 -1.408269) (xy 3.532809 -1.345322) (xy 3.419775 -1.274818)
+				(xy 3.311982 -1.19707) (xy 3.209764 -1.11239) (xy 3.113457 -1.02109) (xy 3.023394 -0.923482) (xy 2.939911 -0.819879)
+				(xy 2.863343 -0.710593) (xy 2.794025 -0.595936) (xy 2.732291 -0.476221) (xy 2.678476 -0.351759)
+				(xy 2.643239 -0.254665) (xy 2.632915 -0.222707) (xy 2.622192 -0.187738) (xy 2.612125 -0.153312)
+				(xy 2.60377 -0.12298) (xy 2.601325 -0.113516) (xy 2.594937 -0.088309) (xy 2.590395 -0.071312) (xy 2.587229 -0.061523)
+				(xy 2.584967 -0.057938) (xy 2.583137 -0.059555) (xy 2.581268 -0.065371) (xy 2.580344 -0.06888) (xy 2.569168 -0.111528)
+				(xy 2.559773 -0.146688) (xy 2.551662 -0.176095) (xy 2.544337 -0.201484) (xy 2.5373 -0.224589) (xy 2.530053 -0.247145)
+				(xy 2.523749 -0.266019) (xy 2.475984 -0.392487) (xy 2.419792 -0.514914) (xy 2.35552 -0.632912) (xy 2.283511 -0.746092)
+				(xy 2.20411 -0.854066) (xy 2.117661 -0.956446) (xy 2.024511 -1.052842) (xy 1.925002 -1.142866) (xy 1.81948 -1.226131)
+				(xy 1.70829 -1.302246) (xy 1.591776 -1.370825) (xy 1.503478 -1.415943) (xy 1.420626 -1.453214) (xy 1.334289 -1.48748)
+				(xy 1.247369 -1.517699) (xy 1.162766 -1.54283) (xy 1.119877 -1.553725) (xy 1.100893 -1.558595) (xy 1.086409 -1.563005)
+				(xy 1.078194 -1.566372) (xy 1.077124 -1.567801) (xy 1.082831 -1.570044) (xy 1.095944 -1.574029)
+				(xy 1.114642 -1.579235) (xy 1.137104 -1.58514) (xy 1.142453 -1.586502) (xy 1.269384 -1.623496) (xy 1.393666 -1.669384)
+				(xy 1.514773 -1.723802) (xy 1.63218 -1.786384) (xy 1.745361 -1.856765) (xy 1.853789 -1.934579) (xy 1.956939 -2.01946)
+				(xy 2.054286 -2.111044) (xy 2.145303 -2.208965) (xy 2.229466 -2.312857) (xy 2.272109 -2.371645)
+				(xy 2.345811 -2.485427) (xy 2.411295 -2.603515) (xy 2.468694 -2.72621) (xy 2.518141 -2.853815) (xy 2.559772 -2.986631)
+				(xy 2.581551 -3.071036) (xy 2.583217 -3.075553)
+			)
+			(stroke
+				(width 0)
+				(type solid)
+			)
+			(fill solid)
+			(layer "F.SilkS")
+		)
+	)
 	(footprint "cipulot_parts:HOLE_M2"
 		(layer "F.Cu")
@@
 	(footprint "LOGO"
 		(layer "B.Cu")
-		(at 246.38 49.065336 180)
+		(at 245.745 48.535428 180)
 		(property "Reference" "G***"
 			(at 0 0 0)
@@
 	)
 	(gr_line
-		(start 255.27 52.599908)
-		(end 255.27 48.789908)
+		(start 254.935 52.07)
+		(end 254.935 48.26)
 		(stroke
 			(width 0.15)
@@
 	)
 	(gr_arc
-		(start 237.09 48.789908)
-		(mid 237.461974 47.891882)
-		(end 238.36 47.519908)
+		(start 236.155 48.26)
+		(mid 236.526972 47.361969)
+		(end 237.425 46.99)
 		(stroke
 			(width 0.15)
@@
 	)
 	(gr_line
-		(start 238.36 53.869908)
-		(end 254 53.869908)
+		(start 237.425 53.34)
+		(end 253.665 53.34)
 		(stroke
 			(width 0.15)
@@
 	)
 	(gr_line
-		(start 254 47.519908)
-		(end 238.36 47.519908)
+		(start 253.665 46.99)
+		(end 237.425 46.99)
 		(stroke
 			(width 0.15)
@@
 	)
 	(gr_arc
-		(start 255.27 52.599908)
-		(mid 254.898026 53.497934)
-		(end 254 53.869908)
+		(start 254.935 52.07)
+		(mid 254.563023 52.96802)
+		(end 253.665 53.34)
 		(stroke
 			(width 0.15)
@@
 	)
 	(gr_arc
-		(start 238.36 53.869908)
-		(mid 237.461974 53.497934)
-		(end 237.09 52.599908)
+		(start 237.425 53.34)
+		(mid 236.526972 52.968026)
+		(end 236.155 52.07)
 		(stroke
 			(width 0.15)
@@
 	)
 	(gr_line
-		(start 237.09 48.789908)
-		(end 237.09 52.599908)
+		(start 236.155 48.26)
+		(end 236.155 52.07)
 		(stroke
 			(width 0.15)
@@
 	)
 	(gr_arc
-		(start 254 47.519908)
-		(mid 254.898026 47.891882)
-		(end 255.27 48.789908)
+		(start 253.665 46.99)
+		(mid 254.563023 47.361975)
+		(end 254.935 48.26)
 		(stroke
 			(width 0.15)
@@
 	)
 	(gr_text "design by xonuss & xezioh"
-		(at 246.18 51.329908 0)
+		(at 245.545 50.8 0)
 		(layer "B.SilkS")
 		(effects
@@
 	)
 	(gr_text "pcb by calvin0563"
-		(at 246.18 52.917408 0)
+		(at 245.545 52.3875 0)
 		(layer "B.SilkS")
 		(effects
@@
 	)
 	(gr_text "EC"
-		(at 238.76 49.204359 0)
+		(at 238.125 48.674451 0)
 		(layer "B.SilkS")
 		(effects
